File: kicad_source/mcp2515.kicad_sch (KiCad schematic)
At the start: 14 parts, among them P5 SM04B-GHS-TB, P6 SM04B-GHS-TB, U2 MCP2515-I/SO, U3 SN65HVD232, Y1 RH100-16.000-16-3030-EXT-TR

Commit message: updated layout
Parts:
- U2: footprint SOIC:SOIC-18_7.5x11.6mm_Pitch1.27mm -> Package_SO:SOIC-18W_7.5x11.6mm_P1.27mm
- U3: footprint SOIC:SOIJ-8_5.3x5.3mm_Pitch1.27mm -> Package_SO:SOIC-8_3.9x4.9mm_P1.27mm
Changed lines of the file:
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@@
     (property "Reference" "U2" (id 0) (at 127 37.465 0))
     (property "Value" "MCP2515-I/SO" (id 1) (at 127 39.7764 0))
-    (property "Footprint" "SOIC:SOIC-18_7.5x11.6mm_Pitch1.27mm" (id 2) (at 127 55.88 0)
+    (property "Footprint" "Package_SO:SOIC-18W_7.5x11.6mm_P1.27mm" (id 2) (at 127 55.88 0)
       (effects (font (size 1.27 1.27)) hide)
     )
@@
       (effects (font (size 1.524 1.524)))
     )
-    (property "Footprint" "SOIC:SOIJ-8_5.3x5.3mm_Pitch1.27mm" (id 2) (at 232.41 67.31 0)
+    (property "Footprint" "Package_SO:SOIC-8_3.9x4.9mm_P1.27mm" (id 2) (at 232.41 67.31 0)
       (effects (font (size 1.524 1.524)) hide)
     )

Commit message: added page with outputs
Other:
- title: OpenCyphalRobotController07 -> CyphalRobotController07/CAN
Changed lines of the file:
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@@
   (paper "A4")
   (title_block
-    (title "OpenCyphalRobotController07")
-    (date "2023-07-24")
+    (title "CyphalRobotController07/CAN")
+    (date "2023-10-01")
     (rev "0.1")
     (company "generationmake")

Commit message: started layout
Parts:
- renumbered P5 to J5, P6 to J6
Changed lines of the file:
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@@
   (symbol (lib_id "Connector_Generic_MountingPin:Conn_01x04_MountingPin") (at 223.52 105.41 0) (unit 1)
     (in_bom yes) (on_board yes)
-    (property "Reference" "P5" (id 0) (at 225.5012 104.3686 0)
+    (property "Reference" "J5" (id 0) (at 225.5012 104.3686 0)
       (effects (font (size 1.27 1.27)) (justify left))
     )
@@
   (symbol (lib_id "Connector_Generic_MountingPin:Conn_01x04_MountingPin") (at 223.52 129.54 0) (unit 1)
     (in_bom yes) (on_board yes)
-    (property "Reference" "P6" (id 0) (at 225.5012 128.4986 0)
+    (property "Reference" "J6" (id 0) (at 225.5012 128.4986 0)
       (effects (font (size 1.27 1.27)) (justify left))
     )

Commit message: made first draft of placement
Parts:
- Y1: footprint crystals:Crystal_SMD_0603_4Pads -> Crystal:Crystal_SMD_3225-4Pin_3.2x2.5mm
Changed lines of the file:
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@@
     (property "Reference" "Y1" (id 0) (at 170.18 75.692 0))
     (property "Value" "RH100-16.000-16-3030-EXT-TR" (id 1) (at 170.18 78.0034 0))
-    (property "Footprint" "crystals:Crystal_SMD_0603_4Pads" (id 2) (at 170.18 86.36 0)
+    (property "Footprint" "Crystal:Crystal_SMD_3225-4Pin_3.2x2.5mm" (id 2) (at 170.18 86.36 0)
       (effects (font (size 1.27 1.27)) hide)
     )

Commit message: made first draft of layout
Parts:
- J5, J6: value SM04B-GHS-TB -> BM04B-GHS-TBT; footprint Connector_JST:JST_GH_SM04B-GHS-TB_1x04-1MP_P1.25mm_Horizontal -> Connector_JST:JST_GH_BM04B-GHS-TBT_1x04-1MP_P1.25mm_Vertical
Changed lines of the file:
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@@
       (effects (font (size 1.27 1.27)) (justify left))
     )
-    (property "Value" "SM04B-GHS-TB" (id 1) (at 225.5012 106.68 0)
+    (property "Value" "BM04B-GHS-TBT" (id 1) (at 225.5012 106.68 0)
       (effects (font (size 1.27 1.27)) (justify left))
     )
-    (property "Footprint" "Connector_JST:JST_GH_SM04B-GHS-TB_1x04-1MP_P1.25mm_Horizontal" (id 2) (at 223.52 105.41 0)
+    (property "Footprint" "Connector_JST:JST_GH_BM04B-GHS-TBT_1x04-1MP_P1.25mm_Vertical" (id 2) (at 223.52 105.41 0)
       (effects (font (size 1.27 1.27)) hide)
     )
@@
       (effects (font (size 1.27 1.27)) (justify left))
     )
-    (property "Value" "SM04B-GHS-TB" (id 1) (at 225.5012 130.81 0)
+    (property "Value" "BM04B-GHS-TBT" (id 1) (at 225.5012 130.81 0)
       (effects (font (size 1.27 1.27)) (justify left))
     )
-    (property "Footprint" "Connector_JST:JST_GH_SM04B-GHS-TB_1x04-1MP_P1.25mm_Horizontal" (id 2) (at 223.52 129.54 0)
+    (property "Footprint" "Connector_JST:JST_GH_BM04B-GHS-TBT_1x04-1MP_P1.25mm_Vertical" (id 2) (at 223.52 129.54 0)
       (effects (font (size 1.27 1.27)) hide)
     )
