File: kicad_source/History.kicad_sch (KiCad schematic)
At the start: 0 parts

Commit message: updated schematic history, updated schematic pdf
Other:
- note added: "0.1"
- note added: "0.2"
- note added: "2023-12-03"
- note added: "2024-01-15"
- note added: "2024-01-21"
- note added: "2024-01-22"
- note added: "added JST XH connector for motor and encoder"
- note added: "added always on connector for +BATT"
- note added: "added level converters on encoder inputs"
- note added: "added protection on CAN"
- note added: "added tvs diode on input"
- note added: "added weak pull down on EM_STOP_D"
- note added: "changed R45 to 1k3"
- note added: "combined 3.3V nets"
- note added: "connected current sense output to analog in of RP2040"
- note added: "replaced INA226 by INA232 to support up to 40V"
- note added: "replaced tantal with electrolytic capacitors"
- note added: "used raspberry pi pico with headers"
- note removed: "1.0"
Changed lines of the file:
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@@
     (company "generationmake")
+  )
+  (text "Bernhard Mayer" (at 58.42 68.58 0)
+    (effects (font (size 1.524 1.524)) (justify left bottom))
+  )
+  (text "2024-01-21" (at 34.29 64.77 0)
+    (effects (font (size 1.524 1.524)) (justify left bottom))
+  )
+  (text "2023-12-03" (at 34.29 45.72 0)
+    (effects (font (size 1.524 1.524)) (justify left bottom))
+  )
+  (text "Bernhard Mayer" (at 58.42 53.34 0)
+    (effects (font (size 1.524 1.524)) (justify left bottom))
+  )
+  (text "Bernhard Mayer" (at 58.42 72.39 0)
+    (effects (font (size 1.524 1.524)) (justify left bottom))
+  )
+  (text "2024-01-21" (at 34.29 53.34 0)
+    (effects (font (size 1.524 1.524)) (justify left bottom))
+  )
+  (text "replaced tantal with electrolytic capacitors" (at 85.09 64.77 0)
+    (effects (font (size 1.524 1.524)) (justify left bottom))
+  )
+  (text "2024-01-22" (at 34.29 68.58 0)
+    (effects (font (size 1.524 1.524)) (justify left bottom))
+  )
+  (text "2023-12-03" (at 34.29 34.29 0)
+    (effects (font (size 1.524 1.524)) (justify left bottom))
+  )
+  (text "Bernhard Mayer" (at 58.42 34.29 0)
+    (effects (font (size 1.524 1.524)) (justify left bottom))
+  )
+  (text "added level converters on encoder inputs" (at 85.09 49.53 0)
+    (effects (font (size 1.524 1.524)) (justify left bottom))
+  )
+  (text "changed R45 to 1k3" (at 85.09 34.29 0)
+    (effects (font (size 1.524 1.524)) (justify left bottom))
+  )
+  (text "replaced INA226 by INA232 to support up to 40V" (at 85.09 68.58 0)
+    (effects (font (size 1.524 1.524)) (justify left bottom))
+  )
+  (text "added protection on CAN" (at 85.09 57.15 0)
+    (effects (font (size 1.524 1.524)) (justify left bottom))
+  )
+  (text "added always on connector for +BATT" (at 85.09 41.91 0)
+    (effects (font (size 1.524 1.524)) (justify left bottom))
+  )
+  (text "2024-01-21" (at 34.29 60.96 0)
+    (effects (font (size 1.524 1.524)) (justify left bottom))
+  )
+  (text "2024-01-22" (at 34.29 72.39 0)
+    (effects (font (size 1.524 1.524)) (justify left bottom))
+  )
+  (text "2023-12-03" (at 34.29 41.91 0)
+    (effects (font (size 1.524 1.524)) (justify left bottom))
+  )
+  (text "added JST XH connector for motor and encoder" (at 85.09 45.72 0)
+    (effects (font (size 1.524 1.524)) (justify left bottom))
+  )
+  (text "Bernhard Mayer" (at 58.42 45.72 0)
+    (effects (font (size 1.524 1.524)) (justify left bottom))
   )
   (text "2023-10-01" (at 34.29 22.86 0)
     (effects (font (size 1.524 1.524)) (justify left bottom))
   )
-  (text "1.0" (at 21.59 22.86 0)
+  (text "Bernhard Mayer" (at 58.42 41.91 0)
+    (effects (font (size 1.524 1.524)) (justify left bottom))
+  )
+  (text "added tvs diode on input" (at 85.09 60.96 0)
+    (effects (font (size 1.524 1.524)) (justify left bottom))
+  )
+  (text "Bernhard Mayer" (at 58.42 57.15 0)
+    (effects (font (size 1.524 1.524)) (justify left bottom))
+  )
+  (text "2023-12-03" (at 34.29 38.1 0)
+    (effects (font (size 1.524 1.524)) (justify left bottom))
+  )
+  (text "Bernhard Mayer" (at 58.42 64.77 0)
+    (effects (font (size 1.524 1.524)) (justify left bottom))
+  )
+  (text "added weak pull down on EM_STOP_D" (at 85.09 38.1 0)
+    (effects (font (size 1.524 1.524)) (justify left bottom))
+  )
+  (text "Bernhard Mayer" (at 58.42 38.1 0)
+    (effects (font (size 1.524 1.524)) (justify left bottom))
+  )
+  (text "used raspberry pi pico with headers" (at 85.09 53.34 0)
+    (effects (font (size 1.524 1.524)) (justify left bottom))
+  )
+  (text "2024-01-21" (at 34.29 57.15 0)
+    (effects (font (size 1.524 1.524)) (justify left bottom))
+  )
+  (text "combined 3.3V nets" (at 85.09 30.48 0)
+    (effects (font (size 1.524 1.524)) (justify left bottom))
+  )
+  (text "2023-12-03" (at 34.29 30.48 0)
+    (effects (font (size 1.524 1.524)) (justify left bottom))
+  )
+  (text "0.2" (at 21.59 30.48 0)
+    (effects (font (size 1.524 1.524)) (justify left bottom))
+  )
+  (text "2024-01-15" (at 34.29 49.53 0)
+    (effects (font (size 1.524 1.524)) (justify left bottom))
+  )
+  (text "0.1" (at 21.59 22.86 0)
+    (effects (font (size 1.524 1.524)) (justify left bottom))
+  )
+  (text "Bernhard Mayer" (at 58.42 49.53 0)
+    (effects (font (size 1.524 1.524)) (justify left bottom))
+  )
+  (text "Bernhard Mayer" (at 58.42 60.96 0)
+    (effects (font (size 1.524 1.524)) (justify left bottom))
+  )
+  (text "connected current sense output to analog in of RP2040"
+    (at 85.09 72.39 0)
     (effects (font (size 1.524 1.524)) (justify left bottom))
   )
@@
     (effects (font (size 1.524 1.524)) (justify left bottom))
   )
+  (text "Bernhard Mayer" (at 58.42 30.48 0)
+    (effects (font (size 1.524 1.524)) (justify left bottom))
+  )
